File: hardware/board-design/board-design.kicad_sch (KiCad schematic)
At the start: 1 part, among them J1 Conn_01x02_Pin

Commit message: feat(schematic): update schematic
Connections:
- no-connect marks 2 -> 1
Other:
- added sheet STM32 (stm32.kicad_sch)
- sheet DC-DC-Buck-Converter ports: added mcu_output; removed mcu_input
- moved on the sheet: J1
